Commit message: my first foxy commit

File: description/gazebo_control.xacro (robot description, xacro)
@@ -19,3 +19,34 @@
         </plugin>
     </gazebo>
+<gazebo reference="rplidar_a1">
+  <sensor type="ray" name="head_hokuyo_sensor">
+    <pose>0 0 0 0 0 0</pose>
+    <visualize>true</visualize>
+    <update_rate>5</update_rate>
+    <ray>
+      <scan>
+        <horizontal>
+          <samples>360</samples>
+          <resolution>1</resolution>
+          <min_angle>4.7</min_angle>
+          <max_angle>7.9</max_angle>
+        </horizontal>
+      </scan>
+      <range>
+        <min>0.120</min>
+        <max>3.5</max>
+        <resolution>0.015</resolution>
+      </range>
+      <noise>
+        <type>gaussian</type>
+        <mean>0.0</mean>
+        <stddev>0.01</stddev>
+      </noise>
+    </ray>
+    <plugin name="gazebo_ros_hokuyo_controller" filename="libgazebo_ros_laser.so">
+      <topicName>scan</topicName>
+      <frameName>rplidar_a1</frameName>
+    </plugin>
+  </sensor>
+</gazebo>
 </robot>

File: description/robot_core.xacro (robot description, xacro)
@@ -121,3 +121,25 @@
         <mu2 value="0.001"/> <!-- (To Be Measured) -->
     </gazebo>
+    <joint name="lidar_a1_joint" type="fixed">
+        <parent link="base_link"/>
+        <child link="lidar_a1"/>
+        <origin xyz="0 0 0.285" rpy="0 0 0" />
+    </joint>
+    <link name="lidar_a1">
+        <visual>
+            <geometry>
+                <mesh filename="file://$(find albot-description)/description/meshes/lidar.stl"/>
+            </geometry>
+            <origin xyz="0 0 -0.025"/>
+        </visual>
+        <collision>
+            <origin xyz="0 0 -0.01"/>
+            <geometry>
+                <mesh filename="file://$(find albot-description)/description/meshes/lidar.stl"/>
+            </geometry>
+        </collision>
+        <xacro:inertial_sphere mass="0.1" radius="0.05"> <!-- mass in kg, length and radius in meters (To Be Measured) -->
+            <origin xyz="0 0 0" rpy="0 0 0"/>
+        </xacro:inertial_sphere>
+    </link>
 </robot>

Commit message: update lidar ROS2 plugin

File: description/gazebo_control.xacro (robot description, xacro)
@@ -9,6 +9,6 @@
             <wheel_diameter>0.08</wheel_diameter>
             <!-- Limits -->
-            <max_wheel_torque>200</max_wheel_torque>
-            <max_wheel_acceleration>10.0</max_wheel_acceleration>
+            <max_wheel_torque>20</max_wheel_torque>
+            <max_wheel_acceleration>1.0</max_wheel_acceleration>
             <!-- Output -->
             <odometry_frame>odom</odometry_frame>
@@ -19,9 +19,9 @@
         </plugin>
     </gazebo>
-<gazebo reference="rplidar_a1">
+<gazebo reference="lidar_a1">
   <sensor type="ray" name="head_hokuyo_sensor">
     <pose>0 0 0 0 0 0</pose>
     <visualize>true</visualize>
-    <update_rate>5</update_rate>
+    <update_rate>10</update_rate>
     <ray>
       <scan>
@@ -29,6 +29,6 @@
           <samples>360</samples>
           <resolution>1</resolution>
-          <min_angle>4.7</min_angle>
-          <max_angle>7.9</max_angle>
+          <min_angle>-3.14</min_angle>
+          <max_angle>3.14</max_angle>
         </horizontal>
       </scan>
@@ -36,5 +36,4 @@
         <min>0.120</min>
         <max>3.5</max>
-        <resolution>0.015</resolution>
       </range>
       <noise>
@@ -44,7 +43,10 @@
       </noise>
     </ray>
-    <plugin name="gazebo_ros_hokuyo_controller" filename="libgazebo_ros_laser.so">
-      <topicName>scan</topicName>
-      <frameName>rplidar_a1</frameName>
+    <plugin name="gazebo_ros_hokuyo_controller" filename="libgazebo_ros_ray_sensor.so">
+      <ros>
+        <argument>~/out:=scan</argument>
+      </ros>
+      <output_type>sensor_msgs/LaserScan</output_type>
+      <frameName>lidar_a1</frameName>
     </plugin>
   </sensor>

File: description/robot_core.xacro (robot description, xacro)
@@ -40,5 +40,5 @@
             </geometry>
         </collision>
-        <xacro:inertial_box mass="3" x="0.455" y="0.4" z="0.263"> <!-- mass in kg, length and radius in meters (To Be Measured) -->
+        <xacro:inertial_box mass="5" x="0.455" y="0.4" z="0.263"> <!-- mass in kg, length and radius in meters (To Be Measured) -->
             <origin xyz="0.183 0 -.1" rpy="0 0 ${pi}"/>
         </xacro:inertial_box>
@@ -113,5 +113,5 @@
             </geometry>
         </collision>
-        <xacro:inertial_sphere mass="0.1" radius="0.05"> <!-- mass in kg, length and radius in meters (To Be Measured) -->
+        <xacro:inertial_sphere mass="5" radius="0.05"> <!-- mass in kg, length and radius in meters (To Be Measured) -->
             <origin xyz="0 0 0" rpy="0 0 0"/>
         </xacro:inertial_sphere>
@@ -124,5 +124,5 @@
         <parent link="base_link"/>
         <child link="lidar_a1"/>
-        <origin xyz="0 0 0.285" rpy="0 0 0" />
+        <origin xyz="0 0 0.3" rpy="0 0 0" />
     </joint>
     <link name="lidar_a1">
@@ -131,5 +131,5 @@
                 <mesh filename="file://$(find albot-description)/description/meshes/lidar.stl"/>
             </geometry>
-            <origin xyz="0 0 -0.025"/>
+            <origin xyz="0 0 -0.04"/>
         </visual>
         <collision>

Commit message: feat(albot-description): add real lidar configs and update chassis mesh

File: description/gazebo_control.xacro (robot description, xacro)
@@ -19,36 +19,3 @@
         </plugin>
     </gazebo>
-<gazebo reference="lidar_a1">
-  <sensor type="ray" name="head_hokuyo_sensor">
-    <pose>0 0 0 0 0 0</pose>
-    <visualize>true</visualize>
-    <update_rate>10</update_rate>
-    <ray>
-      <scan>
-        <horizontal>
-          <samples>360</samples>
-          <resolution>1</resolution>
-          <min_angle>-3.14</min_angle>
-          <max_angle>3.14</max_angle>
-        </horizontal>
-      </scan>
-      <range>
-        <min>0.120</min>
-        <max>3.5</max>
-      </range>
-      <noise>
-        <type>gaussian</type>
-        <mean>0.0</mean>
-        <stddev>0.01</stddev>
-      </noise>
-    </ray>
-    <plugin name="gazebo_ros_hokuyo_controller" filename="libgazebo_ros_ray_sensor.so">
-      <ros>
-        <argument>~/out:=scan</argument>
-      </ros>
-      <output_type>sensor_msgs/LaserScan</output_type>
-      <frameName>lidar_a1</frameName>
-    </plugin>
-  </sensor>
-</gazebo>
 </robot>

File: description/robot_core.xacro (robot description, xacro)
@@ -28,14 +28,14 @@
     <link name="chassis">
         <visual>
-            <origin xyz="0.183 0 -.1" rpy="0 0 ${pi}"/>
+            <origin xyz="0.183 0 -0.02" rpy="0 0 ${pi}"/>
             <geometry>
-                <mesh filename="file://$(find albot-description)/description/meshes/base_link.stl"/>
+                <mesh filename="file://$(find albot-description)/description/meshes/chassis_equiped.stl"/>
             </geometry>
             <material name="white"/>
         </visual>
         <collision>
-            <origin  xyz="0.183 0 -.1" rpy="0 0 ${pi}"/>
+            <origin  xyz="0.183 0 -0.02" rpy="0 0 ${pi}"/>
             <geometry>
-                <mesh filename="file://$(find albot-description)/description/meshes/base_link.stl"/>
+                <mesh filename="file://$(find albot-description)/description/meshes/chassis_equiped.stl"/>
             </geometry>
         </collision>
@@ -121,25 +121,3 @@
         <mu2 value="0.001"/> <!-- (To Be Measured) -->
     </gazebo>
-    <joint name="lidar_a1_joint" type="fixed">
-        <parent link="base_link"/>
-        <child link="lidar_a1"/>
-        <origin xyz="0 0 0.3" rpy="0 0 0" />
-    </joint>
-    <link name="lidar_a1">
-        <visual>
-            <geometry>
-                <mesh filename="file://$(find albot-description)/description/meshes/lidar.stl"/>
-            </geometry>
-            <origin xyz="0 0 -0.04"/>
-        </visual>
-        <collision>
-            <origin xyz="0 0 -0.01"/>
-            <geometry>
-                <mesh filename="file://$(find albot-description)/description/meshes/lidar.stl"/>
-            </geometry>
-        </collision>
-        <xacro:inertial_sphere mass="0.1" radius="0.05"> <!-- mass in kg, length and radius in meters (To Be Measured) -->
-            <origin xyz="0 0 0" rpy="0 0 0"/>
-        </xacro:inertial_sphere>
-    </link>
 </robot>
