Commit message: fix(albot-description): fix lidar collision

File: description/lidar.xacro (robot description, xacro)
@@ -14,5 +14,5 @@
         </visual>
         <collision>
-            <origin xyz="0 0 -0.01"/>
+            <origin xyz="0 0 -0.04"/>
             <geometry>
                 <mesh filename="file://$(find albot-description)/description/meshes/lidar.stl"/>
