Commit message: fix(albot-description): fix sonar bug

File: description/sonar.xacro (robot description, xacro)
@@ -10,5 +10,5 @@
             <visual>
                 <geometry>
-                    <mesh filename="file://$(find albot-description)/description/meshes/sonar.stl" scale="0.001 0.001 0.001"/>
+                    <!-- <mesh filename="file://$(find albot-description)/description/meshes/sonar.stl" scale="0.001 0.001 0.001"/> -->
                 </geometry>
                 <origin xyz="0 -0.023 -0.01" rpy="${pi/2} 0 ${pi/2}"/>
@@ -58,5 +58,5 @@
                 <plugin name="bytes_ultrasound" filename="libgazebo_ros_ray_sensor.so">
                     <ros>
-                        <namespace>distance</namespace>
+                        <namespace>${sonar_prefix}_distance</namespace>
                         <remapping>~/out:=${sonar_prefix}_sonar</remapping>
                     </ros>
